File: Hardware/0. Project/WaterPull/WaterPull.brd (EAGLE design)
At the start: 100.1 x 61.8 mm, 51 parts, among them CN1 USB-B, CN2 127/220VAC, CN3 12V @ 150mA, IC1 7812TV, Q1 16 MHz, Q2 BC817, Q3 BC817, SW1 KY-040, T1 BTB16-800BW, T2 7.5V + 7.5V @ 500mA, U1 EL357N, U2 ATMEGA328P-PU, U3 FT232RL, U4 AM2302 (DHT22), U6 REG1117

Commit message: WIP
Parts:
- CN2: device Instrumentos:AK550/2 -> Instrumentos:AK500/2-H
- CN3: device My-Electromechanicals:CON-2P -> My-Electromechanicals:JST-PH2
- R1: device rcl:AK550/2 -> rcl:AK500/2-H
- moved CN1 26.7 mm to (0.25, 52.7), turned to 0 degrees
- moved U4 8.77 mm to (16.6, 58.8), turned to 0 degrees
- moved R9 8.47 mm to (39.9, 52.0), turned to 0 degrees
- moved D3 4.62 mm to (18.1, 51.7)
- moved R14 4.62 mm to (27.4, 11.1), turned to 90 degrees
- moved SW1 4.43 mm to (13.0, 35.2)
- moved LED2 4.27 mm to (22.4, 53.4)
- moved LED3 4.27 mm to (24.5, 53.4)
- moved C4 4.27 mm to (27.1, 49.6)
- moved R11 4.27 mm to (24.5, 49.6)
- moved U3 4.27 mm to (20.3, 38.8)
- moved R10 4.22 mm to (22.4, 49.6)
- moved R13 2.20 mm to (14.2, 51.6), turned to 270 degrees
- moved LCD1 0.44 mm to (44.9, 2.43), flipped to the top
- turned R12 to 90 degrees
Connections:
- removed net N$38: C11.1, C12.1, IC1.3, U6.3
- new net N$13: BR1.+, C10.1, C9.+, IC1.1
- net 12VDC: now also C11.1, C12.1, CN3.2, IC1.3, U6.3; no longer BR1.+, C10.1, C9.+, CN3.1, IC1.1
- net N$37: now also CN3.1; no longer CN3.2
Routing:
- net 5V: track 63.4 -> 222.7 mm, vias 2 -> 5
- net 12VDC: track 44.4 -> 127.9 mm
- net 1WIRE_TEMPERATURE_SENSOR: track 7.81 -> 61.0 mm, vias 0 -> 1
- net GPIO_ROTARY_ENCODER_SWITCH: track 0.00 -> 50.8 mm
- net I2C_LCD_SCL: track 0.00 -> 50.1 mm, vias 0 -> 1
- net I2C_LCD_SDA: track 0.00 -> 47.3 mm, vias 0 -> 1
- net MCU_RESET: track 2.79 -> 45.3 mm, vias 0 -> 1
- net UART_MCU_RX: track 0.00 -> 41.9 mm, vias 0 -> 1
- net GPIO_BUZZER: track 0.00 -> 41.2 mm, vias 0 -> 1
- net N$13: track 0.00 -> 39.6 mm
- net GPIO_ROTARY_ENCODER_SIGNAL-A: track 18.6 -> 54.2 mm, vias 0 -> 1
- net GPIO_ROTARY_ENCODER_SIGNAL-B: track 8.15 -> 41.6 mm
- net UART_MCU_TX: track 0.36 -> 32.4 mm, vias 0 -> 1
- net N$38: track 29.2 -> 0.00 mm
- net N$33: track 11.8 -> 33.3 mm
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- added copper zone on layer 1, net OV
- added copper zone on layer 16, net OV

Commit message: Schematic 1.0 - DONE
Parts:
- removed R1: 500W, rcl:AK500/2-H
- removed T2: 7.5V + 7.5V @ 500mA, My-Transformers:3PINS
- added CN6: USB-B, My-Connectors:USB-B
- added CN7: 7.5V + 7.5V @ 500mA, My-Transformers:3PINS
- added D4: SS34, My-Diodes:DO214AB
- added Q4: BC817, transistor:SOT23-BEC
- added R15: 3k3, My-RLC:R0805
- CN1: value USB-B -> 127/220VAC; device My-Connectors:USB-B -> Instrumentos:AK500/2-H
- CN2: value 127/220VAC -> 500W; device Instrumentos:AK500/2-H -> rcl:AK500/2-H
- R14, R6, R8: device rcl:R0805 -> My-RLC:R0805
- R7: value 220R -> 330R; device rcl:R0805 -> My-RLC:R0805
- moved CN1 99.9 mm to (88.1, 5.22), turned to 180 degrees
- moved CN2 23.1 mm to (71.9, 5.25)
- moved BR1 3.19 mm to (56.3, 18.5)
- moved LED2 1.17 mm to (22.3, 54.6)
- moved LED3 1.17 mm to (24.4, 54.6)
- moved R6 0.58 mm to (62.4, 14.3)
- moved C1 0.43 mm to (46.2, 32.1)
- moved R5 0.31 mm to (94.4, 22.6)
- moved C9 0.30 mm to (55.6, 34.1)
- renumbered IC1 to U8, LCD1 to CN4, OK1 to U7, U4 to CN5
Connections:
- removed net D10: U2.16
- removed net D11: U2.17
- removed net D12: U2.18
- removed net D13: U2.19
- new net N$14: Q4.B, R15.2
- new net N$15: Q4.C, U7.2
- new net N$16: C13.1, C14.1, D4.A, U6.2, U6.4
- net 0V: now also CN6.4, CN6.M1, CN6.M2, Q4.E; no longer CN1.4, CN1.M1, CN1.M2, U7.2
- net 0VAC: now also CN1.1; no longer R1.1
- net 127VAC: now also CN1.2; no longer CN2.2
- net 5V: now also D4.C, R7.1; no longer C13.1, C14.1, U6.2, U6.4
- net A1: now also CN2.2; no longer R1.2
- net GND1: now also CN7.3; no longer T2.3
- net N$33: now also CN6.2; no longer CN1.2
- net N$34: now also CN6.3; no longer CN1.3
- net N$42: now also CN7.1; no longer T2.1
- net PWM_HEATER: now also R15.1; no longer R7.1
- net VUSB: now also CN6.1; no longer CN1.1
Routing:
- net N$15: track 0.00 -> 42.3 mm, vias 0 -> 3
- net 12VDC: track 127.9 -> 94.7 mm, vias 0 -> 1
- net N$16: track 0.00 -> 24.8 mm
- net PWM_HEATER: track 27.6 -> 3.21 mm, vias 1 -> 0
- net 5V: track 222.7 -> 242.6 mm, vias 5 -> 2
- net 127VAC: track 79.6 -> 61.5 mm
- net UART_MCU_RX: track 41.9 -> 32.5 mm
- net MCU_RESET: track 45.3 -> 36.1 mm
- net N$33: track 33.3 -> 25.5 mm, vias 0 -> 1
- net UART_MCU_TX: track 32.4 -> 24.7 mm
- net GPIO_ROTARY_ENCODER_SWITCH: track 50.8 -> 43.3 mm
- net GPIO_BUZZER: track 41.2 -> 34.8 mm
- net N$34: track 33.9 -> 38.6 mm
- net VUSB: track 14.0 -> 18.2 mm
- net N$14: track 0.00 -> 4.20 mm
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- added copper zone on layer 1, net 0V
- added copper zone on layer 16, net 0V
- removed copper zone on layer 1, net OV
- removed copper zone on layer 16, net OV
Other:
- board size 100.1 x 61.8 mm -> 100 x 62 mm
- board text added: "DISPLAY"
- board text added: "FAN"
- board text added: "HEATER"
- board text added: "INPUT"
- board text added: "SENSOR"
- board text added: "TRANSFORMER"
