File: Hardware/0. Project/WaterPull/WaterPull.sch (EAGLE design)
At the start: 53 parts, among them CN1 USB-B, CN2 127/220VAC, CN3 12V @ 150mA, IC1 7812TV, Q1 16 MHz, Q2 BC817, Q3 BC817, SW1 KY-040, SW2 HH 6T, T1 BTB16-800BW, T2 7.5V + 7.5V @ 500mA, U1 EL357N, U2 ATMEGA328P-PU, U3 FT232RL, U4 AM2302 (DHT22), U6 REG1117

Commit message: WIP
Parts:
- R1: device rcl:R-US_ -> rcl:R-US_KRE
Connections:
- removed net N$38: C11.1, C12.1, IC1.VO, U6.VIN
- new net N$13: BR1.+, C10.1, C9.+, IC1.VI
- net 12VDC: now also C11.1, C12.1, IC1.VO, U6.VIN; no longer BR1.+, C10.1, C9.+, IC1.VI

Commit message: Schematic 1.0 - DONE
Parts:
- removed OK1: MOC3020, optocoupler:MOC3010M
- removed R1: 500W, rcl:R-US_KRE
- added CN6: USB-B, My-Connectors:USB-B
- added D4: SS34, My-Diodes:SS34
- added Q4: BC817, transistor:BC817-16-NPN-SOT23-BEC
- added R15: 3k3, My-RLC:R_0805
- added U7: MOC3020, optocoupler:MOC3010M
- CN1: value USB-B -> 127/220VAC; device My-Connectors:USB-B -> Instrumentos:GENERATOR-FP
- CN2: value 127/220VAC -> 500W; device Instrumentos:GENERATOR-FP -> rcl:R-US_KRE
- R14, R6, R8: device rcl:R-EU_R0805 -> My-RLC:R_0805
- R7: value 220R -> 330R; device rcl:R-EU_R0805 -> My-RLC:R_0805
- renumbered IC1 to U8, LCD1 to CN4, T2 to CN7, U4 to CN5
Connections:
- removed net D10: U2.(SS)PB2
- removed net D11: U2.(MOSI)PB3
- removed net D12: U2.(MISO)PB4
- removed net D13: U2.(SCK)PB5
- new net N$14: Q4.B, R15.2
- new net N$15: Q4.C, U7.C
- new net N$16: C13.1, C14.1, D4.A, U6.VOUT
- net 0V: now also CN6G$1.4, CN6G$2.S1, CN6G$2.S2, Q4.E; no longer CN1G$1.4, CN1G$2.S1, CN1G$2.S2, OK1.C
- net 0VAC: now also CN1.P$2, CN2.1; no longer CN2.P$2, R1.1
- net 127VAC: now also CN1.P$3; no longer CN2.P$3
- net 5V: now also D4.K, R7.1; no longer C13.1, C14.1, U6.VOUT
- net A1: now also CN2.2; no longer R1.2
- net N$1: now also U7.A1; no longer OK1.A1
- net N$10: now also U7.A; no longer OK1.A
- net N$33: now also CN6G$1.2; no longer CN1G$1.2
- net N$34: now also CN6G$1.3; no longer CN1G$1.3
- net N$9: now also U7.A2; no longer OK1.A2
- net PWM_HEATER: now also R15.1; no longer R7.1
- net VUSB: now also CN6G$1.1; no longer CN1G$1.1
Other:
- moved on the sheet: C1, C2, C5, C6, CN2, D1, D2, Q1, R2, R7, R9, T1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

Commit message: Schematic 1.0 preview added
Other:
- note added: "D0"
- note added: "D1"
- moved on the sheet: B1, BR1, C1, C10, C11, C12, C13, C14, C2, C3, C4, C5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
